Commit message: 3 box robot

File: body.urdf (robot description, URDF)
Before this commit: robot robot, 2 links, 1 joints
Links:
- removed link Leg
- added link LegBack, mass 1; collision box size=1 1 1; visual box size=1 1 1
- added link LegFront, mass 1; collision box size=1 1 1; visual box size=1 1 1
Joints:
- removed joint Torso_Leg
- added joint Torso_Leg_B: type revolute, parent Torso, child LegBack, origin xyz=-0.5 0 1 rpy=0 0 0, axis 0 1 0, limit lower=-3.14159 upper=3.14159 effort=0.0 velocity=0.0
- added joint Torso_Leg_F: type revolute, parent Torso, child LegFront, origin xyz=0.5 0 1 rpy=0 0 0, axis 0 1 0, limit lower=-3.14159 upper=3.14159 effort=0.0 velocity=0.0

Commit message: random movement

File: body.urdf (robot description, URDF)
Before this commit: robot robot, 3 links, 2 joints
Links:
- link Torso: mass 1 -> 10

Commit message: added neural network and modified pyrosim

File: body.urdf (robot description, URDF)
Before this commit: robot robot, 3 links, 2 joints
Links:
- link Torso: mass 10 -> 1

Commit message: generate quadruped

File: body.urdf (robot description, URDF)
Before this commit: robot robot, 3 links, 2 joints
Links:
- added link LegLeft, mass 1; collision box size=1 0.2 0.2; visual box size=1 0.2 0.2
- added link LegLowerBack, mass 1; collision box size=0.2 0.2 1; visual box size=0.2 0.2 1
- added link LegLowerFront, mass 1; collision box size=0.2 0.2 1; visual box size=0.2 0.2 1
- added link LegLowerLeft, mass 1; collision box size=0.2 0.2 1; visual box size=0.2 0.2 1
- added link LegLowerRight, mass 1; collision box size=0.2 0.2 1; visual box size=0.2 0.2 1
- added link LegRight, mass 1; collision box size=1 0.2 0.2; visual box size=1 0.2 0.2
- link LegBack: geometry collision box size=0.2 1 0.2; visual box size=0.2 1 0.2
- link LegFront: geometry collision box size=0.2 1 0.2; visual box size=0.2 1 0.2
- link Torso: geometry collision box size=1 1 0.5; visual box size=1 1 0.5
Joints:
- added joint Leg_B_Leg_LB: type revolute, parent LegBack, child LegLowerBack, origin xyz=0 -1 0 rpy=0 0 0, axis 0 1 0, limit lower=-3.14159 upper=3.14159 effort=0.0 velocity=0.0
- added joint Leg_F_Leg_LF: type revolute, parent LegFront, child LegLowerFront, origin xyz=0 1 0 rpy=0 0 0, axis 0 1 0, limit lower=-3.14159 upper=3.14159 effort=0.0 velocity=0.0
- added joint Leg_L_Leg_LL: type revolute, parent LegLeft, child LegLowerLeft, origin xyz=-1 0 0 rpy=0 0 0, axis 1 0 0, limit lower=-3.14159 upper=3.14159 effort=0.0 velocity=0.0
- added joint Leg_R_Leg_LR: type revolute, parent LegRight, child LegLowerRight, origin xyz=1 0 0 rpy=0 0 0, axis 1 0 0, limit lower=-3.14159 upper=3.14159 effort=0.0 velocity=0.0
- added joint Torso_Leg_L: type revolute, parent Torso, child LegLeft, origin xyz=-0.5 0 1 rpy=0 0 0, axis 0 1 0, limit lower=-3.14159 upper=3.14159 effort=0.0 velocity=0.0
- added joint Torso_Leg_R: type revolute, parent Torso, child LegRight, origin xyz=0.5 0 1 rpy=0 0 0, axis 0 1 0, limit lower=-3.14159 upper=3.14159 effort=0.0 velocity=0.0
- joint Torso_Leg_B: axis 0 1 0 -> 1 0 0; origin xyz=-0.5 0 1 rpy=0 0 0 -> xyz=0 -0.5 1 rpy=0 0 0
- joint Torso_Leg_F: axis 0 1 0 -> 1 0 0; origin xyz=0.5 0 1 rpy=0 0 0 -> xyz=0 0.5 1 rpy=0 0 0
